File: hv-probe-passive/hv-probe-passive.kicad_pcb (KiCad board)
At the start: 2 copper layers, 210 x 27 mm, 20 parts, among them J2 OUT

Commit message: added a script for rough estimation of internal capacitance, corrected schematic
Other:
- board text added: "Poliurethane Resin HUNTSMAN CW5620 BLUE eps = 6 dielectric breakdown 25 kV / 1 mm viscosity 1300 mPas"
- board text removed: "Poliurethane Resin HUNTSMAN CW5620 BLUE \eps = 6 dielectric breakdown 25 kV / 1 mm viscosity 1300 mPas"
Changed lines of the file:
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@@
 		)
 	)
-	(gr_text "Poliurethane Resin HUNTSMAN CW5620 BLUE \n\\eps = 6\ndielectric breakdown 25 kV / 1 mm\nviscosity 1300 mPas"
+	(gr_text "Poliurethane Resin HUNTSMAN CW5620 BLUE \neps = 6\ndielectric breakdown 25 kV / 1 mm\nviscosity 1300 mPas"
 		(at 160.75 69.75 0)
 		(layer "Cmts.User")
