File: hv-probe-passive/hv-probe-passive.kicad_pcb (KiCad board)
At the start: 2 copper layers, 210 x 27 mm, 20 parts, among them J2 OUT

Commit message: cleaned up the schematic and readme
Routing:
- net Net-(C12-Pad2): track 62.4 -> 61.7 mm
Other:
- outline, holes or cut-outs redrawn
- board text added: "JSK 2026"
- board text removed: "JSK 2024"
