File: hv-probe-passive/hv-probe-passive.kicad_sch (KiCad schematic)
At the start: 20 parts, among them J2 OUT

Commit message: added a script for rough estimation of internal capacitance, corrected schematic
Parts:
- C1, C10, C11, C12, C2, C3, C4, C5, C8, C9: value 47p -> 24p
Changed lines of the file:
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@@
 		)
 	)
-	(text_box "in the original build a resin with \\eps of ~4-5 was used, i have resin with \\eps = 6 i magnified the capacitances."
+	(text_box "in the original build a resin with eps of ~4-5 was used, so since i have resin with eps = 6 i magnified the capacitances."
 		(exclude_from_sim no)
 		(at 91.44 110.49 0)
@@
 			)
 		)
-		(property "Value" "47p"
+		(property "Value" "24p"
 			(at 91.4463 42.545 90)
 			(effects
@@
 			)
 		)
-		(property "Value" "47p"
+		(property "Value" "24p"
 			(at 157.4863 42.545 90)
 			(effects
@@
 			)
 		)
-		(property "Value" "47p"
+		(property "Value" "24p"
 			(at 151.1363 42.545 90)
 			(effects
@@
 			)
 		)
-		(property "Value" "47p"
+		(property "Value" "24p"
 			(at 124.4663 42.545 90)
 			(effects
@@
 			)
 		)
-		(property "Value" "47p"
+		(property "Value" "24p"
 			(at 107.9563 42.545 90)
 			(effects
@@
 			)
 		)
-		(property "Value" "47p"
+		(property "Value" "24p"
 			(at 85.0963 42.545 90)
 			(effects
@@
 			)
 		)
-		(property "Value" "47p"
+		(property "Value" "24p"
 			(at 134.6263 42.545 90)
 			(effects
@@
 			)
 		)
-		(property "Value" "47p"
+		(property "Value" "24p"
 			(at 118.1163 42.545 90)
 			(effects
@@
 			)
 		)
-		(property "Value" "47p"
+		(property "Value" "24p"
 			(at 140.9763 42.545 90)
 			(effects
@@
 			)
 		)
-		(property "Value" "47p"
+		(property "Value" "24p"
 			(at 101.6063 42.545 90)
 			(effects
